File: hw2/HW2/HW2.sch (EAGLE design)
At the start: 22 parts, among them J1 USB-MB-H

Commit message: Working on .brd
Parts:
- C5, C6: device HW2:CPOL-USETR2 -> HW2:CPOL-USB45181A
Connections:
- net B3: now also U$2.7.B3; no longer U$2.70.B3
Changed lines of the file:
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@@
 <part name="C3" library="HW2" deviceset="C-US" device="025-024X044" value="0.1uF"/>
 <part name="C4" library="HW2" deviceset="C-US" device="025-024X044" value="0.1uF"/>
-<part name="C5" library="HW2" deviceset="CPOL-US" device="ETR2" value="10uF"/>
-<part name="C6" library="HW2" deviceset="CPOL-US" device="ETR2" value="10uF"/>
+<part name="C5" library="HW2" deviceset="CPOL-US" device="B45181A" value="10uF"/>
+<part name="C6" library="HW2" deviceset="CPOL-US" device="B45181A" value="10uF"/>
 <part name="LED1" library="HW2" deviceset="LED" device="3MM" value="red"/>
 <part name="LED2" library="HW2" deviceset="LED" device="3MM" value="green"/>
@@
 <net name="B3" class="0">
 <segment>
-<pinref part="U$2" gate="G$1" pin="70.B3"/>
+<pinref part="U$2" gate="G$1" pin="7.B3"/>
 <wire x1="-20.32" y1="0" x2="-33.02" y2="0" width="0.1524" layer="91"/>
 <label x="-33.02" y="0" size="1.778" layer="95"/>

Commit message: Finished .brd wiring
Parts:
- J2: device HW2:M05PTH -> HW2:M06SILK_FEMALE_PTH
Changed lines of the file:
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@@
 <part name="J3" library="HW2" deviceset="M08" device="SILK_FEMALE_PTH"/>
 <part name="J4" library="HW2" deviceset="M08" device="SILK_FEMALE_PTH"/>
-<part name="J2" library="HW2" deviceset="M05" device="PTH"/>
+<part name="J2" library="HW2" deviceset="M06" device="SILK_FEMALE_PTH"/>
 <part name="RESET" library="HW2" deviceset="EVQ11" device=""/>
 <part name="USER" library="HW2" deviceset="EVQ11" device=""/>
@@
 <segment>
 <pinref part="J2" gate="G$1" pin="1"/>
-<wire x1="-55.88" y1="35.56" x2="-48.26" y2="35.56" width="0.1524" layer="91"/>
+<wire x1="-58.42" y1="35.56" x2="-48.26" y2="35.56" width="0.1524" layer="91"/>
 <label x="-50.8" y="35.56" size="1.778" layer="95"/>
 </segment>
@@
 <segment>
 <pinref part="J2" gate="G$1" pin="4"/>
-<wire x1="-55.88" y1="43.18" x2="-48.26" y2="43.18" width="0.1524" layer="91"/>
+<wire x1="-58.42" y1="43.18" x2="-48.26" y2="43.18" width="0.1524" layer="91"/>
 <label x="-50.8" y="43.18" size="1.778" layer="95"/>
 </segment>
@@
 <segment>
 <pinref part="J2" gate="G$1" pin="5"/>
-<wire x1="-55.88" y1="45.72" x2="-48.26" y2="45.72" width="0.1524" layer="91"/>
+<wire x1="-58.42" y1="45.72" x2="-48.26" y2="45.72" width="0.1524" layer="91"/>
 <label x="-50.8" y="45.72" size="1.778" layer="95"/>
 </segment>
@@
 <pinref part="J2" gate="G$1" pin="3"/>
 <pinref part="GND14" gate="1" pin="GND"/>
-<wire x1="-55.88" y1="40.64" x2="-35.56" y2="40.64" width="0.1524" layer="91"/>
+<wire x1="-58.42" y1="40.64" x2="-35.56" y2="40.64" width="0.1524" layer="91"/>
 </segment>
 <segment>
@@
 <pinref part="J2" gate="G$1" pin="2"/>
 <pinref part="+3V4" gate="G$1" pin="+3V3"/>
-<wire x1="-55.88" y1="38.1" x2="-43.18" y2="38.1" width="0.1524" layer="91"/>
-</segment>
-<segment>
+<wire x1="-58.42" y1="38.1" x2="-43.18" y2="38.1" width="0.1524" layer="91"/>
+</segment>
+<segment>
